File: Hardware/kiss_sdr_r2/kiss_sdr_r2.kicad_pcb (KiCad board)
At the start: 2 copper layers, 100.4 x 45.7 mm, 76 parts, among them J1 SMA, J2 I_Q_Output, J3 SDR_CLK, J4 +5V, Q1 MMBT3904, U1 OPA2356xxD, U2 SN74CBT3253, U3 74LC74, U4 74AHCT1G04

Commit message: update current files
Parts:
- removed the C16 at (107.7, 92.1)
- removed the C24 at (108.5, 101.4)
- removed the D2 at (91.5, 90.8)
- removed H1: MountingHole_Pad, MountingHole:MountingHole_2.7mm_M2.5_ISO14580_Pad
- removed I_SIG1: I_SIG, TestPoint:TestPoint_THTPad_D2.0mm_Drill1.0mm
- removed J3: SDR_CLK, Connector_PinHeader_2.54mm:PinHeader_1x02_P2.54mm_Vertical
- removed Q1: MMBT3904, Package_TO_SOT_SMD:SOT-23
- removed Q_SIG1: Q_SIG, TestPoint:TestPoint_THTPad_D2.0mm_Drill1.0mm
- removed the R4 at (118.5, 99.2)
- removed the R9 at (122.7, 102.5)
- added +5V1: +5V, TestPoint:TestPoint_THTPad_D2.0mm_Drill1.0mm, F.Cu at (159.3, 112.3)
- added C17: 10uF, Capacitor_SMD:C_0805_2012Metric_Pad1.18x1.45mm_HandSolder, F.Cu at (147.8, 78.6)
- added C3: 0.1uF, Capacitor_SMD:C_0805_2012Metric_Pad1.18x1.45mm_HandSolder, F.Cu at (170.3, 106.6)
- added C6: 912pF, Capacitor_SMD:C_0805_2012Metric_Pad1.18x1.45mm_HandSolder, F.Cu at (104.0, 84.1)
- added C7: 10uF, Capacitor_SMD:C_0805_2012Metric_Pad1.18x1.45mm_HandSolder, F.Cu at (164.5, 106.6)
- added FB1: FerriteBead, 6A 1 9mΩ 33Ω@100MHz ±25% 1206 Ferrite Beads RO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, Inductor_SMD:L_1206_3216Metric_Pad1.42x1.75mm_HandSolder, F.Cu at (125.5, 80.1)
- added L2: 0.185uH, Inductor_SMD:L_1206_3216Metric_Pad1.22x1.90mm_HandSolder, F.Cu at (98.3, 85.0)
- added Q2: J310, Package_TO_SOT_SMD:SOT-23, F.Cu at (111.8, 89.4)
- added Q3: AO3401A, Package_TO_SOT_SMD:SOT-23, F.Cu at (172.6, 102.1)
- added R1: 100R, Resistor_SMD:R_0805_2012Metric_Pad1.20x1.40mm_HandSolder, F.Cu at (124.6, 114.9)
- added R12: 10R, Resistor_SMD:R_0805_2012Metric_Pad1.20x1.40mm_HandSolder, F.Cu at (155.8, 79.8)
- added R15: 0R, Resistor_SMD:R_0805_2012Metric_Pad1.20x1.40mm_HandSolder, F.Cu at (174.8, 113.8)
- added R16: 0R, Resistor_SMD:R_0805_2012Metric_Pad1.20x1.40mm_HandSolder, F.Cu at (171.5, 113.8)
- added R17: 0R, Resistor_SMD:R_0805_2012Metric_Pad1.20x1.40mm_HandSolder, F.Cu at (168.3, 113.8)
- added R3: 10K, Resistor_SMD:R_0805_2012Metric_Pad1.20x1.40mm_HandSolder, F.Cu at (172.3, 98.3)
- added R7: 100K, Resistor_SMD:R_0805_2012Metric_Pad1.20x1.40mm_HandSolder, F.Cu at (115.4, 85.0)
- added U4: OPA2356xxD, Package_SO:SOIC-8_3.9x4.9mm_P1.27mm, F.Cu at (154.1, 83.7)
- added U6: SI5351, jerrys_Library:SI5351_Brd_fp, F.Cu at (181.4, 116.8)
- added sig2: filter1, TestPoint:TestPoint_THTPad_D2.0mm_Drill1.0mm, F.Cu at (95.5, 80.3)
- added sig3: filter_gnd1, TestPoint:TestPoint_THTPad_D2.0mm_Drill1.0mm, F.Cu at (117.3, 114.3)
- added sig4: filter_gnd2, TestPoint:TestPoint_THTPad_D2.0mm_Drill1.0mm, F.Cu at (117.5, 118.8)
- added sig5: filter2, TestPoint:TestPoint_THTPad_D2.0mm_Drill1.0mm, F.Cu at (105.3, 79.3)
- C1: renamed from C23; footprint Capacitor_SMD:C_1206_3216Metric_Pad1.33x1.80mm_HandSolder -> Capacitor_SMD:C_0805_2012Metric_Pad1.18x1.45mm_HandSolder
- C10: renamed from C13; value 0.1F -> 0.1uF; footprint Capacitor_SMD:C_1206_3216Metric_Pad1.33x1.80mm_HandSolder -> Capacitor_SMD:C_0805_2012Metric_Pad1.18x1.45mm_HandSolder
- C11: renamed from C25; footprint Capacitor_SMD:C_1206_3216Metric_Pad1.33x1.80mm_HandSolder -> Capacitor_SMD:C_0805_2012Metric_Pad1.18x1.45mm_HandSolder
- C12: renamed from C19; footprint Capacitor_SMD:C_1206_3216Metric_Pad1.33x1.80mm_HandSolder -> Capacitor_SMD:C_0805_2012Metric_Pad1.18x1.45mm_HandSolder
- C13: renamed from C1; footprint Capacitor_SMD:C_1206_3216Metric_Pad1.33x1.80mm_HandSolder -> Capacitor_SMD:C_0805_2012Metric_Pad1.18x1.45mm_HandSolder
- C14: renamed from C26; footprint Capacitor_SMD:C_1206_3216Metric_Pad1.33x1.80mm_HandSolder -> Capacitor_SMD:C_0805_2012Metric_Pad1.18x1.45mm_HandSolder
- C15: value 130pF -> 0.1uF; footprint Capacitor_SMD:C_1206_3216Metric_Pad1.33x1.80mm_HandSolder -> Capacitor_SMD:C_0805_2012Metric_Pad1.18x1.45mm_HandSolder
- C16: renamed from C2; footprint Capacitor_SMD:C_1206_3216Metric_Pad1.33x1.80mm_HandSolder -> Capacitor_SMD:C_0805_2012Metric_Pad1.18x1.45mm_HandSolder
- C18: renamed from C3; footprint Capacitor_SMD:C_1206_3216Metric_Pad1.33x1.80mm_HandSolder -> Capacitor_SMD:C_0805_2012Metric_Pad1.18x1.45mm_HandSolder
- C19: renamed from C5; value 0.1F -> 0.1uF; footprint Capacitor_SMD:C_1206_3216Metric_Pad1.33x1.80mm_HandSolder -> Capacitor_SMD:C_0805_2012Metric_Pad1.18x1.45mm_HandSolder
- C2: renamed from C11; value 4.7nF -> 1.1nF; footprint Capacitor_SMD:C_1206_3216Metric_Pad1.33x1.80mm_HandSolder -> Capacitor_SMD:C_0805_2012Metric_Pad1.18x1.45mm_HandSolder
- C20: renamed from C6; value 0.1F -> 0.1uF; footprint Capacitor_SMD:C_1206_3216Metric_Pad1.33x1.80mm_HandSolder -> Capacitor_SMD:C_0805_2012Metric_Pad1.18x1.45mm_HandSolder
- C21: renamed from C9; footprint Capacitor_SMD:C_1206_3216Metric_Pad1.33x1.80mm_HandSolder -> Capacitor_SMD:C_0805_2012Metric_Pad1.18x1.45mm_HandSolder
- C22: renamed from C20; footprint Capacitor_SMD:C_1206_3216Metric_Pad1.33x1.80mm_HandSolder -> Capacitor_SMD:C_0805_2012Metric_Pad1.18x1.45mm_HandSolder
- C23: renamed from C21; footprint Capacitor_SMD:C_1206_3216Metric_Pad1.33x1.80mm_HandSolder -> Capacitor_SMD:C_0805_2012Metric_Pad1.18x1.45mm_HandSolder
- C24: renamed from C10; footprint Capacitor_SMD:C_1206_3216Metric_Pad1.33x1.80mm_HandSolder -> Capacitor_SMD:C_0805_2012Metric_Pad1.18x1.45mm_HandSolder
- C25: renamed from C14; footprint Capacitor_SMD:C_1206_3216Metric_Pad1.33x1.80mm_HandSolder -> Capacitor_SMD:C_0805_2012Metric_Pad1.18x1.45mm_HandSolder
- C26: renamed from C4; footprint Capacitor_SMD:C_1206_3216Metric_Pad1.33x1.80mm_HandSolder -> Capacitor_SMD:C_0805_2012Metric_Pad1.18x1.45mm_HandSolder
- C27: renamed from C7; footprint Capacitor_SMD:C_1206_3216Metric_Pad1.33x1.80mm_HandSolder -> Capacitor_SMD:C_0805_2012Metric_Pad1.18x1.45mm_HandSolder
- C28: renamed from C18; footprint Capacitor_SMD:C_1206_3216Metric_Pad1.33x1.80mm_HandSolder -> Capacitor_SMD:C_0805_2012Metric_Pad1.18x1.45mm_HandSolder
- C4: renamed from C12; value 4.7nF -> 1.1nF; footprint Capacitor_SMD:C_1206_3216Metric_Pad1.33x1.80mm_HandSolder -> Capacitor_SMD:C_0805_2012Metric_Pad1.18x1.45mm_HandSolder
- C5: renamed from C22; footprint Capacitor_SMD:C_1206_3216Metric_Pad1.33x1.80mm_HandSolder -> Capacitor_SMD:C_0805_2012Metric_Pad1.18x1.45mm_HandSolder
- C8: value 0.1F -> 66.6pF; footprint Capacitor_SMD:C_1206_3216Metric_Pad1.33x1.80mm_HandSolder -> Capacitor_SMD:C_0805_2012Metric_Pad1.18x1.45mm_HandSolder
- C9: renamed from C17; value 130pF -> 912pF; footprint Capacitor_SMD:C_1206_3216Metric_Pad1.33x1.80mm_HandSolder -> Capacitor_SMD:C_0805_2012Metric_Pad1.18x1.45mm_HandSolder
- D1: value BAT43 -> BAV99; footprint Diode_SMD:D_SOD-123 -> Package_TO_SOT_SMD:SOT-23
- J1: value SMA -> pwr; footprint Connector_Coaxial:SMA_Samtec_SMA-J-P-X-ST-EM1_EdgeMount -> Connector_PinHeader_2.54mm:PinHeader_1x04_P2.54mm_Vertical
- J2: value I_Q_Output -> SMA; footprint Connector_PinHeader_2.54mm:PinHeader_1x03_P2.54mm_Vertical -> Connector_Coaxial:SMA_Samtec_SMA-J-P-X-ST-EM1_EdgeMount
- J4: value +5V -> Audio Out; footprint Connector_PinHeader_2.54mm:PinHeader_1x02_P2.54mm_Vertical -> Connector_Audio:Jack_3.5mm_CUI_SJ-3523-SMT_Horizontal
- L1: renamed from L3; value 10uH -> 2.5uH; footprint Capacitor_SMD:C_1210_3225Metric_Pad1.33x2.70mm_HandSolder -> Inductor_SMD:L_1206_3216Metric_Pad1.22x1.90mm_HandSolder
- L3: renamed from L1; value 10uH -> 2.54uH; footprint Resistor_SMD:R_1210_3225Metric_Pad1.30x2.65mm_HandSolder -> Inductor_SMD:L_1206_3216Metric_Pad1.22x1.90mm_HandSolder
- L4: renamed from L2; value 10uH -> 0.185uH; footprint Resistor_SMD:R_1210_3225Metric_Pad1.30x2.65mm_HandSolder -> Inductor_SMD:L_1206_3216Metric_Pad1.22x1.90mm_HandSolder
- R10: renamed from R16; footprint Resistor_SMD:R_1206_3216Metric_Pad1.30x1.75mm_HandSolder -> Resistor_SMD:R_0805_2012Metric_Pad1.20x1.40mm_HandSolder
- R11: renamed from R17; footprint Resistor_SMD:R_1206_3216Metric_Pad1.30x1.75mm_HandSolder -> Resistor_SMD:R_0805_2012Metric_Pad1.20x1.40mm_HandSolder
- R13: renamed from R1; footprint Resistor_SMD:R_1206_3216Metric_Pad1.30x1.75mm_HandSolder -> Resistor_SMD:R_0805_2012Metric_Pad1.20x1.40mm_HandSolder
- R14: renamed from R3; footprint Resistor_SMD:R_1206_3216Metric_Pad1.30x1.75mm_HandSolder -> Resistor_SMD:R_0805_2012Metric_Pad1.20x1.40mm_HandSolder
- R18: renamed from R6; value 10K -> 100R; footprint Resistor_SMD:R_1206_3216Metric_Pad1.30x1.75mm_HandSolder -> Resistor_SMD:R_0805_2012Metric_Pad1.20x1.40mm_HandSolder
- R19: renamed from R8; value 10K -> 100R; footprint Resistor_SMD:R_1206_3216Metric_Pad1.30x1.75mm_HandSolder -> Resistor_SMD:R_0805_2012Metric_Pad1.20x1.40mm_HandSolder
- R2: value 2.7K -> 100K; footprint Resistor_SMD:R_1206_3216Metric_Pad1.30x1.75mm_HandSolder -> Resistor_SMD:R_0805_2012Metric_Pad1.20x1.40mm_HandSolder
- R20: renamed from R12; value 10K -> 100R; footprint Resistor_SMD:R_1206_3216Metric_Pad1.30x1.75mm_HandSolder -> Resistor_SMD:R_0805_2012Metric_Pad1.20x1.40mm_HandSolder
- R21: renamed from R14; value 10K -> 100R; footprint Resistor_SMD:R_1206_3216Metric_Pad1.30x1.75mm_HandSolder -> Resistor_SMD:R_0805_2012Metric_Pad1.20x1.40mm_HandSolder
- R22: renamed from R10; footprint Resistor_SMD:R_1206_3216Metric_Pad1.30x1.75mm_HandSolder -> Resistor_SMD:R_0805_2012Metric_Pad1.20x1.40mm_HandSolder
- R23: renamed from R5; footprint Resistor_SMD:R_1206_3216Metric_Pad1.30x1.75mm_HandSolder -> Resistor_SMD:R_0805_2012Metric_Pad1.20x1.40mm_HandSolder
- R24: renamed from R7; footprint Resistor_SMD:R_1206_3216Metric_Pad1.30x1.75mm_HandSolder -> Resistor_SMD:R_0805_2012Metric_Pad1.20x1.40mm_HandSolder
- R25: renamed from R13; footprint Resistor_SMD:R_1206_3216Metric_Pad1.30x1.75mm_HandSolder -> Resistor_SMD:R_0805_2012Metric_Pad1.20x1.40mm_HandSolder
- R4: renamed from R18; footprint Resistor_SMD:R_1206_3216Metric_Pad1.30x1.75mm_HandSolder -> Resistor_SMD:R_0805_2012Metric_Pad1.20x1.40mm_HandSolder
- R5: renamed from R19; footprint Resistor_SMD:R_1206_3216Metric_Pad1.30x1.75mm_HandSolder -> Resistor_SMD:R_0805_2012Metric_Pad1.20x1.40mm_HandSolder
- R6: renamed from R20; footprint Resistor_SMD:R_1206_3216Metric_Pad1.30x1.75mm_HandSolder -> Resistor_SMD:R_0805_2012Metric_Pad1.20x1.40mm_HandSolder
- R8: renamed from R11; value 10R -> 27R; footprint Resistor_SMD:R_1206_3216Metric_Pad1.30x1.75mm_HandSolder -> Resistor_SMD:R_0805_2012Metric_Pad1.20x1.40mm_HandSolder
- R9: renamed from R15; value 68R -> 27R; footprint Resistor_SMD:R_1206_3216Metric_Pad1.30x1.75mm_HandSolder -> Resistor_SMD:R_0805_2012Metric_Pad1.20x1.40mm_HandSolder
- U1: value OPA2356xxD -> LD1117S50TR_SOT223; footprint Package_SO:SOIC-8W_5.3x5.3mm_P1.27mm -> Package_TO_SOT_SMD:SOT-223-3_TabPin2
- moved J1 97.0 mm to (179.3, 105.6), turned to 180 degrees
- moved J2 96.4 mm to (84.3, 87.8), turned to -90 degrees
- moved GND3 78.9 mm to (98.0, 119.1)
- moved GND1 63.5 mm to (104.1, 119.9)
- moved R2 56.6 mm to (173.8, 106.1), turned to -90 degrees
- moved CLK1 51.5 mm to (134.3, 117.8)
- moved C15 50.0 mm to (151.8, 78.8), turned to 180 degrees
- moved C1 38.4 mm to (128.6, 114.9)
- moved C5 38.2 mm to (128.6, 108.3)
- moved R4 38.1 mm to (128.6, 110.5)
- moved R5 37.9 mm to (128.6, 112.7)
- moved U2 37.2 mm to (133.3, 114.2)
- moved C14 37.2 mm to (134.0, 109.6)
- moved U3 34.7 mm to (141.1, 111.0)
- moved J4 34.6 mm to (173.3, 89.8), turned to -90 degrees
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- renumbered D3 to D2, FB1 to FB2, GND3 to GND2, GND2 to GND3, U4 to U2, U2 to U5
Connections:
- C1 pad 1: Net-(J3-Pin_2) -> /SMP_CLK
- C10 pad 1: Net-(Q1-B) -> Net-(Q2-G)
- C10 pad 2: Net-(C13-Pad2) -> Net-(C10-Pad2)
- C13 pad 2: +5V -> Net-(C13-Pad2)
- C15 pad 1: Net-(C12-Pad1) -> Net-(U4C-V+)
- C2 pad 2: Net-(D1-K) -> Net-(J2-In)
- C25 pad 1: Net-(U1B--) -> Net-(U4B--)
- C25 pad 2: Net-(C14-Pad2) -> Net-(C25-Pad2)
- C26 pad 1: Net-(U1A--) -> Net-(U4A--)
- C26 pad 2: Net-(C4-Pad2) -> Net-(C26-Pad2)
- C27 pad 2: Net-(J2-Pin_3) -> Net-(C27-Pad2)
- C28 pad 2: Net-(J2-Pin_2) -> Net-(C28-Pad2)
- C4 pad 1: Net-(C12-Pad1) -> Net-(C4-Pad1)
- C8 pad 1: Net-(Q1-C) -> Net-(C8-Pad1)
- C8 pad 2: Net-(C8-Pad2) -> Net-(C10-Pad2)
- C9 pad 1: Net-(C13-Pad2) -> Net-(C10-Pad2)
- CLK1 pad 1: Net-(J3-Pin_2) -> Net-(U3A-C)
- D1 pad 1: Net-(D1-K) -> GND
- J1 pad 1: Net-(D1-K) -> GND
- J1 pad 2: GND -> Net-(J1-Pin_2)
- J2 pad 1: GND -> Net-(J2-In)
- J2 pad 2: Net-(J2-Pin_2) -> GND
- L3 pad 1: Net-(C12-Pad1) -> Net-(C4-Pad1)
- L3 pad 2: Net-(C16-Pad1) -> Net-(C8-Pad1)
- L4 pad 1: Net-(C16-Pad1) -> GND
- L4 pad 2: Net-(C13-Pad2) -> Net-(C10-Pad2)
- R13 pad 2: +5V -> Net-(C13-Pad2)
- R18 pad 2: Net-(U1A-+) -> Net-(U4A-+)
- R19 pad 2: Net-(U1A--) -> Net-(U4A--)
- R2 pad 1: Net-(Q1-B) -> Net-(J1-Pin_2)
- R2 pad 2: +5V -> GND
- R20 pad 2: Net-(U1B-+) -> Net-(U4B-+)
- R21 pad 2: Net-(U1B--) -> Net-(U4B--)
- R22 pad 1: Net-(U1B--) -> Net-(U4B--)
- R22 pad 2: Net-(C14-Pad2) -> Net-(C25-Pad2)
- R23 pad 1: Net-(U1A--) -> Net-(U4A--)
- R23 pad 2: Net-(C4-Pad2) -> Net-(C26-Pad2)
- R24 pad 1: Net-(C4-Pad2) -> Net-(C26-Pad2)
- R25 pad 1: Net-(C14-Pad2) -> Net-(C25-Pad2)
- TR1 pad 1: +5V -> Net-(C13-Pad2)
- TR1 pad 3: Net-(Q1-C) -> Net-(Q2-D)
- U1 pad 1: Net-(C4-Pad2) -> GND
- U1 pad 2: Net-(U1A--) -> +5V
- U1 pad 3: Net-(U1A-+) -> Net-(Q3-S)
- sig1 pad 1: Net-(D1-K) -> Net-(J2-In)
Routing:
- net /SMP_CLK: track 0.00 -> 55.4 mm
- net Net-(C26-Pad2): track 0.00 -> 29.2 mm, vias 0 -> 2
- net /SDA: track 0.00 -> 27.8 mm
- net /SCL: track 0.00 -> 24.8 mm
- net Net-(C4-Pad2): track 24.8 -> 0.00 mm, vias 2 -> 0
- net /CLK_RX_I: track 44.4 -> 25.7 mm, vias 4 -> 2
- net Net-(Q1-B): track 18.3 -> 0.00 mm
- net Net-(D1-K): track 17.8 -> 0.00 mm
- net Net-(Q1-C): track 17.5 -> 0.00 mm
- net Net-(C10-Pad2): track 0.00 -> 17.5 mm
- net Net-(J2-In): track 0.00 -> 16.1 mm
- net GND: track 4.97 -> 19.8 mm, vias 38 -> 78
- net Net-(C28-Pad2): track 0.00 -> 14.8 mm
- net Net-(C4-Pad1): track 0.00 -> 12.9 mm
- net Net-(U1B--): track 12.7 -> 0.00 mm
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Other:
- board text added: "4/4/24"
- board text added: "5V"
- board text added: "GND"
- board text added: "SCL"
- board text added: "SDA"
- board text added: "kiss_sdr, rev0.2"
- board text removed: "+5V"
- board text removed: "3/15/24"
- board text removed: "kiss_sdr, rev0.1"
